File: kicad/usb2mdjoy/usb2mdjoy.kicad_sch (KiCad schematic)
At the start: 7 parts, among them J1 DE9_Socket, J2 UART, U1 RaspberryPi_Pico, U2 FXMA108

Commit message: Split firmware by target, note config-only UF2 in GUI
- firmware/ split into firmware/MSX/ and firmware/MD/
- Stop tracking firmware/pintest_pico.uf2 (debug-only; build from tools/pintest/)
- Config GUI: show that the exported/written UF2 holds settings only
- Docs: AE-LLCNV8-DIP20 module already has C1/C2/R1 on board

Co-Authored-By: Claude Opus 5.5 <noreply@anthropic.com>
Other:
- note added: "ファームウェア: firmware/MD/usb2mdjoy_pico_fxma108.uf2"
- note removed: "ファームウェア: firmware/usb2mdjoy_pico_fxma108.uf2"
Changed lines of the file:
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@@
 		(rev "1")
 		(comment 1 "Raspberry Pi Pico + FXMA108 level translator")
-		(comment 2 "firmware: firmware/usb2mdjoy_pico_fxma108.uf2")
+		(comment 2 "firmware: firmware/MD/usb2mdjoy_pico_fxma108.uf2")
 	)
 	(symbol
@@
 		(instances
 			(project "usb2mdjoy"
-				(path "/aaa00728-68ba-4686-9c9a-408c3db1791a"
+				(path "/223d46f3-7e45-4cae-95a3-4bbc83d8cf3b"
 					(reference "U1")
 					(unit 1)
@@
 		(instances
 			(project "usb2mdjoy"
-				(path "/aaa00728-68ba-4686-9c9a-408c3db1791a"
+				(path "/223d46f3-7e45-4cae-95a3-4bbc83d8cf3b"
 					(reference "U2")
 					(unit 1)
@@
 		(instances
 			(project "usb2mdjoy"
-				(path "/aaa00728-68ba-4686-9c9a-408c3db1791a"
+				(path "/223d46f3-7e45-4cae-95a3-4bbc83d8cf3b"
 					(reference "J1")
 					(unit 1)
@@
 		(instances
 			(project "usb2mdjoy"
-				(path "/aaa00728-68ba-4686-9c9a-408c3db1791a"
+				(path "/223d46f3-7e45-4cae-95a3-4bbc83d8cf3b"
 					(reference "#PWR01")
 					(unit 1)
@@
 		(instances
 			(project "usb2mdjoy"
-				(path "/aaa00728-68ba-4686-9c9a-408c3db1791a"
+				(path "/223d46f3-7e45-4cae-95a3-4bbc83d8cf3b"
 					(reference "#PWR02")
 					(unit 1)
@@
 		(instances
 			(project "usb2mdjoy"
-				(path "/aaa00728-68ba-4686-9c9a-408c3db1791a"
+				(path "/223d46f3-7e45-4cae-95a3-4bbc83d8cf3b"
 					(reference "#PWR03")
 					(unit 1)
@@
 		(instances
 			(project "usb2mdjoy"
-				(path "/aaa00728-68ba-4686-9c9a-408c3db1791a"
+				(path "/223d46f3-7e45-4cae-95a3-4bbc83d8cf3b"
 					(reference "#PWR04")
 					(unit 1)
@@
 		(instances
 			(project "usb2mdjoy"
-				(path "/aaa00728-68ba-4686-9c9a-408c3db1791a"
+				(path "/223d46f3-7e45-4cae-95a3-4bbc83d8cf3b"
 					(reference "#PWR05")
 					(unit 1)
@@
 		(instances
 			(project "usb2mdjoy"
-				(path "/aaa00728-68ba-4686-9c9a-408c3db1791a"
+				(path "/223d46f3-7e45-4cae-95a3-4bbc83d8cf3b"
 					(reference "#PWR06")
 					(unit 1)
@@
 		(instances
 			(project "usb2mdjoy"
-				(path "/aaa00728-68ba-4686-9c9a-408c3db1791a"
+				(path "/223d46f3-7e45-4cae-95a3-4bbc83d8cf3b"
 					(reference "#PWR07")
 					(unit 1)
@@
 		(instances
 			(project "usb2mdjoy"
-				(path "/aaa00728-68ba-4686-9c9a-408c3db1791a"
+				(path "/223d46f3-7e45-4cae-95a3-4bbc83d8cf3b"
 					(reference "#PWR08")
 					(unit 1)
@@
 		(instances
 			(project "usb2mdjoy"
-				(path "/aaa00728-68ba-4686-9c9a-408c3db1791a"
+				(path "/223d46f3-7e45-4cae-95a3-4bbc83d8cf3b"
 					(reference "C1")
 					(unit 1)
@@
 		(instances
 			(project "usb2mdjoy"
-				(path "/aaa00728-68ba-4686-9c9a-408c3db1791a"
+				(path "/223d46f3-7e45-4cae-95a3-4bbc83d8cf3b"
 					(reference "#PWR09")
 					(unit 1)
@@
 		(instances
 			(project "usb2mdjoy"
-				(path "/aaa00728-68ba-4686-9c9a-408c3db1791a"
+				(path "/223d46f3-7e45-4cae-95a3-4bbc83d8cf3b"
 					(reference "#PWR10")
 					(unit 1)
@@
 		(instances
 			(project "usb2mdjoy"
-				(path "/aaa00728-68ba-4686-9c9a-408c3db1791a"
+				(path "/223d46f3-7e45-4cae-95a3-4bbc83d8cf3b"
 					(reference "C2")
 					(unit 1)
@@
 		(instances
 			(project "usb2mdjoy"
-				(path "/aaa00728-68ba-4686-9c9a-408c3db1791a"
+				(path "/223d46f3-7e45-4cae-95a3-4bbc83d8cf3b"
 					(reference "#PWR11")
 					(unit 1)
@@
 		(instances
 			(project "usb2mdjoy"
-				(path "/aaa00728-68ba-4686-9c9a-408c3db1791a"
+				(path "/223d46f3-7e45-4cae-95a3-4bbc83d8cf3b"
 					(reference "#PWR12")
 					(unit 1)
@@
 		(instances
 			(project "usb2mdjoy"
-				(path "/aaa00728-68ba-4686-9c9a-408c3db1791a"
+				(path "/223d46f3-7e45-4cae-95a3-4bbc83d8cf3b"
 					(reference "R1")
 					(unit 1)
@@
 		(instances
 			(project "usb2mdjoy"
-				(path "/aaa00728-68ba-4686-9c9a-408c3db1791a"
+				(path "/223d46f3-7e45-4cae-95a3-4bbc83d8cf3b"
 					(reference "#PWR13")
 					(unit 1)
@@
 		(instances
 			(project "usb2mdjoy"
-				(path "/aaa00728-68ba-4686-9c9a-408c3db1791a"
+				(path "/223d46f3-7e45-4cae-95a3-4bbc83d8cf3b"
 					(reference "J2")
 					(unit 1)
@@
 		(instances
 			(project "usb2mdjoy"
-				(path "/aaa00728-68ba-4686-9c9a-408c3db1791a"
+				(path "/223d46f3-7e45-4cae-95a3-4bbc83d8cf3b"
 					(reference "#PWR14")
 					(unit 1)
@@
 		)
 	)
-	(text "ファームウェア: firmware/usb2mdjoy_pico_fxma108.uf2"
+	(text "ファームウェア: firmware/MD/usb2mdjoy_pico_fxma108.uf2"
 		(exclude_from_sim no)
 		(at 20.32 190.5 0)
