File: kicad/usb2msxjoy/usb2msxjoy.kicad_sch (KiCad schematic)
At the start: 7 parts, among them J1 DE9_Socket, J2 UART, U1 RaspberryPi_Pico, U2 FXMA108

Commit message: Split firmware by target, note config-only UF2 in GUI
- firmware/ split into firmware/MSX/ and firmware/MD/
- Stop tracking firmware/pintest_pico.uf2 (debug-only; build from tools/pintest/)
- Config GUI: show that the exported/written UF2 holds settings only
- Docs: AE-LLCNV8-DIP20 module already has C1/C2/R1 on board

Co-Authored-By: Claude Opus 5.5 <noreply@anthropic.com>
Other:
- note added: "ファームウェア: firmware/MSX/usb2msxjoy_pico_fxma108.uf2"
- note removed: "ファームウェア: firmware/usb2msxjoy_pico_fxma108.uf2"
Changed lines of the file:
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@@
 		(rev "1")
 		(comment 1 "Raspberry Pi Pico + FXMA108 level translator")
-		(comment 2 "firmware: firmware/usb2msxjoy_pico_fxma108.uf2")
+		(comment 2 "firmware: firmware/MSX/usb2msxjoy_pico_fxma108.uf2")
 	)
 	(symbol
@@
 		(instances
 			(project "usb2msxjoy"
-				(path "/57b004bb-6792-43cb-9c7b-e6e5babb1f68"
+				(path "/14e0d3be-1630-47cb-9c3e-8db23d639c9c"
 					(reference "U1")
 					(unit 1)
@@
 		(instances
 			(project "usb2msxjoy"
-				(path "/57b004bb-6792-43cb-9c7b-e6e5babb1f68"
+				(path "/14e0d3be-1630-47cb-9c3e-8db23d639c9c"
 					(reference "U2")
 					(unit 1)
@@
 		(instances
 			(project "usb2msxjoy"
-				(path "/57b004bb-6792-43cb-9c7b-e6e5babb1f68"
+				(path "/14e0d3be-1630-47cb-9c3e-8db23d639c9c"
 					(reference "J1")
 					(unit 1)
@@
 		(instances
 			(project "usb2msxjoy"
-				(path "/57b004bb-6792-43cb-9c7b-e6e5babb1f68"
+				(path "/14e0d3be-1630-47cb-9c3e-8db23d639c9c"
 					(reference "#PWR01")
 					(unit 1)
@@
 		(instances
 			(project "usb2msxjoy"
-				(path "/57b004bb-6792-43cb-9c7b-e6e5babb1f68"
+				(path "/14e0d3be-1630-47cb-9c3e-8db23d639c9c"
 					(reference "#PWR02")
 					(unit 1)
@@
 		(instances
 			(project "usb2msxjoy"
-				(path "/57b004bb-6792-43cb-9c7b-e6e5babb1f68"
+				(path "/14e0d3be-1630-47cb-9c3e-8db23d639c9c"
 					(reference "#PWR03")
 					(unit 1)
@@
 		(instances
 			(project "usb2msxjoy"
-				(path "/57b004bb-6792-43cb-9c7b-e6e5babb1f68"
+				(path "/14e0d3be-1630-47cb-9c3e-8db23d639c9c"
 					(reference "#PWR04")
 					(unit 1)
@@
 		(instances
 			(project "usb2msxjoy"
-				(path "/57b004bb-6792-43cb-9c7b-e6e5babb1f68"
+				(path "/14e0d3be-1630-47cb-9c3e-8db23d639c9c"
 					(reference "#PWR05")
 					(unit 1)
@@
 		(instances
 			(project "usb2msxjoy"
-				(path "/57b004bb-6792-43cb-9c7b-e6e5babb1f68"
+				(path "/14e0d3be-1630-47cb-9c3e-8db23d639c9c"
 					(reference "#PWR06")
 					(unit 1)
@@
 		(instances
 			(project "usb2msxjoy"
-				(path "/57b004bb-6792-43cb-9c7b-e6e5babb1f68"
+				(path "/14e0d3be-1630-47cb-9c3e-8db23d639c9c"
 					(reference "#PWR07")
 					(unit 1)
@@
 		(instances
 			(project "usb2msxjoy"
-				(path "/57b004bb-6792-43cb-9c7b-e6e5babb1f68"
+				(path "/14e0d3be-1630-47cb-9c3e-8db23d639c9c"
 					(reference "#PWR08")
 					(unit 1)
@@
 		(instances
 			(project "usb2msxjoy"
-				(path "/57b004bb-6792-43cb-9c7b-e6e5babb1f68"
+				(path "/14e0d3be-1630-47cb-9c3e-8db23d639c9c"
 					(reference "C1")
 					(unit 1)
@@
 		(instances
 			(project "usb2msxjoy"
-				(path "/57b004bb-6792-43cb-9c7b-e6e5babb1f68"
+				(path "/14e0d3be-1630-47cb-9c3e-8db23d639c9c"
 					(reference "#PWR09")
 					(unit 1)
@@
 		(instances
 			(project "usb2msxjoy"
-				(path "/57b004bb-6792-43cb-9c7b-e6e5babb1f68"
+				(path "/14e0d3be-1630-47cb-9c3e-8db23d639c9c"
 					(reference "#PWR10")
 					(unit 1)
@@
 		(instances
 			(project "usb2msxjoy"
-				(path "/57b004bb-6792-43cb-9c7b-e6e5babb1f68"
+				(path "/14e0d3be-1630-47cb-9c3e-8db23d639c9c"
 					(reference "C2")
 					(unit 1)
@@
 		(instances
 			(project "usb2msxjoy"
-				(path "/57b004bb-6792-43cb-9c7b-e6e5babb1f68"
+				(path "/14e0d3be-1630-47cb-9c3e-8db23d639c9c"
 					(reference "#PWR11")
 					(unit 1)
@@
 		(instances
 			(project "usb2msxjoy"
-				(path "/57b004bb-6792-43cb-9c7b-e6e5babb1f68"
+				(path "/14e0d3be-1630-47cb-9c3e-8db23d639c9c"
 					(reference "#PWR12")
 					(unit 1)
@@
 		(instances
 			(project "usb2msxjoy"
-				(path "/57b004bb-6792-43cb-9c7b-e6e5babb1f68"
+				(path "/14e0d3be-1630-47cb-9c3e-8db23d639c9c"
 					(reference "R1")
 					(unit 1)
@@
 		(instances
 			(project "usb2msxjoy"
-				(path "/57b004bb-6792-43cb-9c7b-e6e5babb1f68"
+				(path "/14e0d3be-1630-47cb-9c3e-8db23d639c9c"
 					(reference "#PWR13")
 					(unit 1)
@@
 		(instances
 			(project "usb2msxjoy"
-				(path "/57b004bb-6792-43cb-9c7b-e6e5babb1f68"
+				(path "/14e0d3be-1630-47cb-9c3e-8db23d639c9c"
 					(reference "J2")
 					(unit 1)
@@
 		(instances
 			(project "usb2msxjoy"
-				(path "/57b004bb-6792-43cb-9c7b-e6e5babb1f68"
+				(path "/14e0d3be-1630-47cb-9c3e-8db23d639c9c"
 					(reference "#PWR14")
 					(unit 1)
@@
 		)
 	)
-	(text "ファームウェア: firmware/usb2msxjoy_pico_fxma108.uf2"
+	(text "ファームウェア: firmware/MSX/usb2msxjoy_pico_fxma108.uf2"
 		(exclude_from_sim no)
 		(at 20.32 186.69 0)
